File: Assignment.kicad_sch (KiCad schematic)
At the start: 10 parts, among them J1 USB_C_Receptacle_PowerOnly_6P, J2 Conn_01x02_Pin

Commit message: Final submission
Parts:
- C1, C2: footprint (none) -> Capacitor_THT:C_Disc_D5.0mm_W2.5mm_P2.50mm
- D1, D2: footprint (none) -> LED_THT:LED_D5.0mm
- J1: footprint (none) -> Connector_USB:USB_C_Receptacle_HRO_TYPE-C-31-M-12
- J2: footprint (none) -> Connector_PinHeader_2.54mm:PinHeader_1x02_P2.54mm_Vertical
- R1, R2, R3: footprint (none) -> Resistor_THT:R_Axial_DIN0207_L6.3mm_D2.5mm_P7.62mm_Horizontal
- TP1: footprint (none) -> Package_SO:SOIC-8_3.9x4.9mm_P1.27mm
Changed lines of the file:
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@@
 (kicad_sch
-	(version 20231120)
+	(version 20250114)
 	(generator "eeschema")
-	(generator_version "8.0")
+	(generator_version "9.0")
 	(paper "A4")
+	(rectangle
+		(start 99.06 46.99)
+		(end 177.8 100.33)
+		(stroke
+			(width 0.254)
+			(type dash)
+		)
+		(fill
+			(type none)
+		)
+	)
+	(rectangle
+		(start 209.55 91.44)
+		(end 245.11 114.3)
+		(stroke
+			(width 0.4)
+			(type dash)
+		)
+		(fill
+			(type none)
+		)
+	)
+	(rectangle
+		(start 184.15 30.48)
+		(end 240.03 77.47)
+		(stroke
+			(width 0.254)
+			(type dash)
+		)
+		(fill
+			(type none)
+		)
+	)
+	(text "Battery Charger Circuit\n"
+		(exclude_from_sim no)
+		(at 138.938 43.688 0)
+		(effects
+			(font
+				(size 1.27 1.27)
+			)
+		)
+	)
+	(text "Battery Connector\n"
+		(exclude_from_sim no)
+		(at 227.076 89.154 0)
+		(effects
+			(font
+				(size 1.27 1.27)
+			)
+		)
+	)
+	(text "Type C \n"
+		(exclude_from_sim no)
+		(at 212.09 28.194 0)
+		(effects
+			(font
+				(size 1.27 1.27)
+			)
+		)
+	)
 	(junction
 		(at 133.35 69.85)
@@
 		)
 	)
-	(rectangle
-		(start 99.06 46.99)
-		(end 177.8 100.33)
-		(stroke
-			(width 0.254)
-			(type dash)
-		)
-		(fill
-			(type none)
-		)
-	)
-	(rectangle
-		(start 209.55 91.44)
-		(end 245.11 114.3)
-		(stroke
-			(width 0.4)
-			(type dash)
-		)
-		(fill
-			(type none)
-		)
-	)
-	(rectangle
-		(start 184.15 30.48)
-		(end 240.03 77.47)
-		(stroke
-			(width 0.254)
-			(type dash)
-		)
-		(fill
-			(type none)
-		)
-	)
-	(text "Battery Charger Circuit\n"
-		(exclude_from_sim no)
-		(at 138.938 43.688 0)
-		(effects
-			(font
-				(size 1.27 1.27)
-			)
-		)
-	)
-	(text "Battery Connector\n"
-		(exclude_from_sim no)
-		(at 227.076 89.154 0)
-		(effects
-			(font
-				(size 1.27 1.27)
-			)
-		)
-	)
-	(text "Type C \n"
-		(exclude_from_sim no)
-		(at 212.09 28.194 0)
-		(effects
-			(font
-				(size 1.27 1.27)
-			)
-		)
-	)
 	(symbol
 		(lib_id "power:VD")
@@
 			)
 		)
-		(property "Footprint" ""
+		(property "Footprint" "LED_THT:LED_D5.0mm"
 			(at 125.73 77.47 0)
 			(effects
@@
 			)
 		)
-		(property "Footprint" ""
+		(property "Footprint" "Resistor_THT:R_Axial_DIN0207_L6.3mm_D2.5mm_P7.62mm_Horizontal"
 			(at 149.352 86.36 90)
 			(effects
@@
 			)
 		)
-		(property "Footprint" ""
+		(property "Footprint" "Connector_PinHeader_2.54mm:PinHeader_1x02_P2.54mm_Vertical"
 			(at 222.25 101.6 0)
 			(effects
@@
 			)
 		)
-		(property "Footprint" ""
+		(property "Footprint" "Resistor_THT:R_Axial_DIN0207_L6.3mm_D2.5mm_P7.62mm_Horizontal"
 			(at 123.952 85.09 90)
 			(effects
@@
 			)
 		)
-		(property "Footprint" ""
+		(property "Footprint" "Capacitor_THT:C_Disc_D5.0mm_W2.5mm_P2.50mm"
 			(at 107.6452 78.74 0)
 			(effects
@@
 		(on_board yes)
 		(dnp no)
-		(fields_autoplaced yes)
 		(property "Reference" "TP1"
 			(at 144.4341 63.5 0)
@@
 			)
 		)
-		(property "Footprint" ""
+		(property "Footprint" "Package_SO:SOIC-8_3.9x4.9mm_P1.27mm"
 			(at 142.24 77.47 0)
 			(effects
@@
 			)
 		)
-		(property "Footprint" ""
+		(property "Footprint" "LED_THT:LED_D5.0mm"
 			(at 116.84 77.47 0)
 			(effects
@@
 			)
 		)
-		(property "Footprint" ""
+		(property "Footprint" "Connector_USB:USB_C_Receptacle_HRO_TYPE-C-31-M-12"
 			(at 213.36 50.8 0)
 			(effects
@@
 			)
 		)
-		(property "Footprint" ""
+		(property "Footprint" "Resistor_THT:R_Axial_DIN0207_L6.3mm_D2.5mm_P7.62mm_Horizontal"
 			(at 115.062 85.09 90)
 			(effects
@@
 			)
 		)
-		(property "Footprint" ""
+		(property "Footprint" "Capacitor_THT:C_Disc_D5.0mm_W2.5mm_P2.50mm"
 			(at 166.0652 77.47 0)
 			(effects
@@
 		)
 	)
+	(embedded_fonts no)
 )
